Commit message: Modify BERNARD model paths, and enhance reward functions for reinforcement learning

File: source/bernard/bernard/data/bernard/urdf/bernard.urdf (robot description, URDF)
Before this commit: robot bernard, 9 links, 8 joints
Links:
- link body: geometry collision box size=0.1180978 0.2033129 0.10758; visual mesh filename=meshes/ESWITCH_TL3301SPF160QGBLK_Varsay_01_ESWITCH_TL3301SP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 scale=1. 1. 1.
- link l_arm: geometry collision box size=0.0455878 0.1951695 0.0850000; visual mesh filename=meshes/ak60_6/body_ak60_6.obj scale=1. 1. 1.
- link l_foot: geometry collision box size=0.037 0.1267169 0.0110000; visual mesh filename=meshes/l_foot_Foot_New_1_Foot_New_1.obj scale=1. 1. 1.
- link l_forearm: geometry collision box size=0.0174227 0.0454954 0.186567; visual mesh filename=meshes/bearing28x8/forearm_bearing_12x28x8mm__2x28x8mm_Bear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 scale=1. 1. 1.
- link r_arm: geometry collision box size=0.0455878 0.1951695 0.0850000; visual mesh filename=meshes/ak60_6/body_ak60_6.obj scale=1. 1. 1.
- link r_foot: geometry collision box size=0.037 0.1267169 0.0110000; visual mesh filename=meshes/r_foot_Foot_New_1_Foot_New_1.obj scale=1. 1. 1.
- link r_forearm: geometry collision box size=0.0174227 0.0454954 0.186567; visual mesh filename=meshes/bearing28x8/forearm_bearing_12x28x8mm__2x28x8mm_Bear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 scale=1. 1. 1.
