Commit message: Add HiL script and tweak locomotion env

File: BERNARD/urdf/BERNARD.urdf (robot description, URDF)
Before this commit: robot BERNARD, 9 links, 8 joints
Links:
- removed link l_arm
- removed link r_arm
- added link l_thigh, mass 0.85000; collision box size=0.10532 0.04085 0.20466; visual mesh filename=../meshes/obj/L_Arm.obj scale=1.00000 1.00000 1.00000
- added link r_thigh, mass 0.85000; collision box size=0.10532 0.04085 0.20466; visual mesh filename=../meshes/obj/R_Arm.obj scale=1.00000 1.00000 1.00000
Joints:
- removed joint l_arm_joint
- removed joint l_hip_joint
- removed joint r_arm_joint
- removed joint r_hip_joint
- added joint l_hip1_joint: type revolute, parent body, child l_hip, origin xyz=0.04683 0.04994 -0.02923 rpy=0.00000 0.00000 0.00000, axis 1.00000 0.00000 0.00000, limit lower=-0.52360 upper=0.52360 effort=9.00000 velocity=9.00000
- added joint l_hip2_joint: type revolute, parent l_hip, child l_thigh, origin xyz=-0.04685 0.05205 -0.00010 rpy=0.00000 0.00000 0.00000, axis 0.00000 1.00000 0.00000, limit lower=-0.87266 upper=1.57080 effort=9.00000 velocity=9.00000
- added joint r_hip1_joint: type revolute, parent body, child r_hip, origin xyz=0.04683 -0.04994 -0.02923 rpy=0.00000 0.00000 0.00000, axis 1.00000 0.00000 0.00000, limit lower=-0.52360 upper=0.52360 effort=9.00000 velocity=9.00000
- added joint r_hip2_joint: type revolute, parent r_hip, child r_thigh, origin xyz=-0.04685 -0.05206 -0.00010 rpy=0.00000 0.00000 0.00000, axis 0.00000 -1.00000 0.00000, limit lower=-1.57080 upper=0.87266 effort=9.00000 velocity=9.00000
- joint l_knee_joint: parent l_arm -> l_thigh
- joint r_knee_joint: parent r_arm -> r_thigh
